File: SmallAvionic/Joyce/Joyce.kicad_sch (KiCad schematic)
At the start: 34 parts, among them IC1 BMP390, J1 QWIIC_RIGHT_ANGLE, J2 CONN_01_1MM, J4 CONN_01_1MM, U1 STM32F103C8Tx, U4 MMC5983MA_QFN16, U5 W25Q128JVE

Commit message: joyce push
Parts:
- added BMP390: ~, symbol New_Library:BMP390
- added C (x2): 100nf, symbol Device:C
Connections:
- net CLK is gone; now on net SPI2_SCK: U5.6 (CLK)
- net DI is gone; now on net SPI2_MOSI: U5.5 (DI/IO_{0})
- net DO is gone; now on net SPI2_MISO: U5.2 (DO/IO_{1})
- net GNDREF is gone; now on net GND: C1.2, C2.2, C4.2, D3.1 (K), U2.4 (GNDA), U2.6 (GNDIO), U3.3 (GND), U5.4 (GND)
- net INT A is gone; now on net INT2_A: JP3.1 (A)
- net SCK_3V is gone; now on net SPI1_SCK: IC1.2 (SCK)
- net SCK/SCL is gone; now on net SPI1_SCK: U2.8 (SCx)
- net SCL is gone; now on net I2C1_SCL: J1.4, R3.1, TP3.1, U4.1 (SCL/SCK)
- net SDA is gone; now on net I2C1_SDA: J1.3, R2.1, TP2.1, U4.16 (SDA/SDI)
- net SDI_3V is gone; now on net SPI1_MOSI: IC1.4 (SDI)
- net SDI/SDA is gone; now on net SPI1_MOSI: U2.9 (SDx)
- net SDO is gone; now on net SPI1_MISO: U2.10 (SDO2), U2.15 (SDO1)
- net SDO/ADR is gone; now on net SPI1_MISO: IC1.5 (SDO), R4.1, SJ1.1
- net VCC is gone; now on net VDD_2: C4.1, R5.2, U5.3 (~{WP}/IO_{2}), U5.7 (~{HOLD}/~{RESET}/IO_{3}), U5.8 (VCC)
- net VDD is gone; now on net VDD_1: JP2.2 (B)
- net CS_3V: no longer IC1.6 (CSB)
- net GND: now also U1.23 (VSS), U1.35 (VSS), U1.47 (VSS), BMP390.3 (V_SS), BMP390.8 (V_SS), BMP390.9 (V_SS), C.2, C.2
- net INT: now also BMP390.7 (INT); no longer IC1.7 (INT)
- net LDO_3V3: now reaches U1.1 (VBAT)
- net INT_1: now reaches U1.10 (PA0)
- net INT_1: now also IC1.7 (INT)
- net SPI1_NSS: now reaches U1.14 (PA4)
- net SPI1_NSS: now also D2.C, IC1.6 (CSB), U2.14 (CSB1), BMP390.6 (CSB)
- net SPI1_SCK: now reaches U1.15 (PA5)
- net SPI1_SCK: now also BMP390.2 (SCK)
- net SPI1_MISO: now reaches U1.16 (PA6)
- net SPI1_MISO: now also BMP390.5 (SDO)
- net SPI1_MOSI: now reaches U1.17 (PA7)
- net SPI1_MOSI: now also BMP390.4 (SDI)
- net VDD_1: now reaches U1.24 (VDD)
- net VDD_1: now also IC1.1 (VDDIO), IC1.10 (VDD), R1.2, R4.2, BMP390.1 (V_DDIO), BMP390.10 (V_DD), C.1, C.1
- net SPI2_NSS: now reaches U1.25 (PB12)
- net SPI2_NSS: now also U5.1 (~{CS})
- net SPI2_SCK: now reaches U1.26 (PB13)
- net SPI2_MISO: now reaches U1.27 (PB14)
- net SPI2_MOSI: now reaches U1.28 (PB15)
- net UART1_TX: now reaches U1.30 (PA9)
- net UART1_RX: now reaches U1.31 (PA10)
- net UART1_CTS: now reaches U1.32 (PA11)
- net UART1_RTS: now reaches U1.33 (PA12)
- net VDD_2: now reaches U1.36 (VDD)
- net I2C1_SCL: now reaches U1.42 (PB6)
- net I2C1_SDA: now reaches U1.43 (PB7)
- net VDD_3: now reaches U1.48 (VDD)
- net VDD_3: now also C3.1, I2C_PU0.2, J1.2, R2.2, R7.2, TP1.1, U4.13 (VDDIO), U4.2 (VDD)
- removed net 3.3V: C3.1, I2C_PU0.2, IC1.1 (VDDIO), IC1.10 (VDD), J1.2, R1.2, R2.2, R4.2, R7.2, TP1.1, U4.13 (VDDIO), U4.2 (VDD)
- removed net CS: D2.C, U2.14 (CSB1), U5.1 (~{CS})
Other:
- moved on the sheet: D2, R1, R4, R7, SJ1
