File: SmallAvionic/Ray/Ray.kicad_sch (KiCad schematic)
At the start: 12 parts, among them U1 STM32F103C8Tx, U2 BMI088

Commit message: Ray finish IMU,BMP, Madnetometer. But just whatever3 7 21 copy from internet
Parts:
- removed D1, D2, D3: 1N4007, Diode_THT:D_DO-41_SOD81_P10.16mm_Horizontal, symbol Diode:1N4007
- added C, C10, C11, C8, C9: 10uF, symbol Device:C
- added C2, C5, C6, C7: C, symbol Device:C
- added D1, D3: LED, symbol Device:LED
- added D2: 1N4148, Diode_THT:D_DO-35_SOD27_P7.62mm_Horizontal, symbol Diode:1N4148
- added Q1, Q2: NMOS, symbol Simulation_SPICE:NMOS
- added Q3, Q4: BSS138, Package_TO_SOT_SMD:SOT-23, symbol Transistor_FET:BSS138
- added R10, R11, R5, R6, R7, R8, R9: 10K, symbol Device:R
- added R12: 100K, symbol Device:R
- added R13: 1K, symbol Device:R
- added U3: AP2112K-3.3, Package_TO_SOT_SMD:SOT-23-5, symbol Regulator_Linear:AP2112K-3.3
- added U4: XC6206PxxxMR, Package_TO_SOT_SMD:SOT-23-3, symbol Regulator_Linear:XC6206PxxxMR
- R1: renamed from R2; value R -> 4.7K
- R2: renamed from R1; value R -> 4.7K
- R3, R4: value R -> 4.7K
Connections:
- net GND: now also C.2, C10.2, C11.2, C2.2, C5.2, C6.2, C7.2, C8.2, C9.2, D1.1 (K), D3.1 (K), U3.2 (GND), U4.1 (GND)
- net SCL_3v3: now also R2.2, Q1.3 (S)
- net SDA_3v3: now also R3.2, Q2.3 (S)
- net VCC: now reaches R4.1
- net VCC: now also R1.1, C.1, C2.1, C5.1, R6.1, R7.1, U4.3 (VI)
- net SDA: now reaches R4.2
- net SDA: now also R3.1, Q2.1 (D), Q2.2 (G)
- net SCL: now reaches R1.2
- net SCL: now also R2.1, Q1.1 (D), Q1.2 (G)
- new net: C6.1, C7.1, U4.2 (VO)
- new net: D2.2 (A), R10.2
- new net: D3.2 (A), R13.2
- new net: D1.2 (A), R5.2
- new net 3v3: C11.1, C8.1, C9.1, Q3.1 (G), Q4.1 (G), R10.1, R11.1, R12.1, R13.1, R5.1, R8.1, R9.1, U3.3 (EN), U3.5 (VOUT)
- new net CAP: C10.1
- new net CS: D2.1 (K)
- new net SCK_3V: Q4.3 (D), R8.2
- new net SCK/SCL: Q4.2 (S), R6.2
- new net SDI_3V': Q3.3 (D), R9.2
- new net SDI/SDA: Q3.2 (S), R7.2
- new net SDO/ADR: R11.2, R12.2
- no-connect marks 1 -> 2
Other:
- note added: "LEVEL SHIFTING (5V <--> 3V)"
- note added: "MMC5983MA_QFN16"
- note added: "Magnetometer - MMC5983MA_QFN16"
- note added: "VDD 2.8~3.6 V VDDIO 2.8~3.6V I2C address : 0x30"
- note added: "Ｆor SOI set CSB low at startup DD=MISO, SDI=MOSI,SCK=SCK, CSB=CS/SSEL For IC leave CSB pulled high (default value) SDI=SDA, SCK=SCL"
- moved on the sheet: C1, C3, R1, R2, R3, R4, U1, U2

Commit message: Ray copy finish internet For SMALLAvionic. It might not work success T_T
Parts:
- added C12, C13, C14, C15: 10uF, symbol Device:C
- added L1: L, symbol Device:L
- added R14, R15: 2.2k, symbol Device:R
- added R16, R17, R18, R19, R20, R21: 4.7K, symbol Device:R
- added U5: W25Q128JVS, Package_SO:SOIC-8_5.3x5.3mm_P1.27mm, symbol Memory_Flash:W25Q128JVS
- added U6: W25Q128JVE, Package_SON:WSON-8-1EP_8x6mm_P1.27mm_EP3.4x4.3mm, symbol Memory_Flash:W25Q128JVE
- added U7: TPS62142, Package_DFN_QFN:VQFN-16-1EP_3x3mm_P0.5mm_EP1.68x1.68mm_ThermalVias, symbol Regulator_Switching:TPS62142
Connections:
- net GND is gone; now on net 3v3: C.2, C1.2, C10.2, C11.2, C2.2, C3.2, C5.2, C6.2, C7.2, C8.2, C9.2, D1.1 (K), D3.1 (K), U2.2 (GNDA), U2.4 (GNDA), U2.6 (GNDIO), U3.2 (GND), U4.1 (GND)
- net SDA is gone; now on net SCL: Q2.1 (D), Q2.2 (G), R3.1, R4.2
- net SDI/SDA is gone; now on net CS: Q3.2 (S), R7.2
- net VCC is gone; now on net 3v3: C.1, C2.1, C5.1, R1.1, R4.1, R6.1, R7.1, U4.3 (VI)
- net 3v3: now also C12.1, C12.2, C13.1, C13.2, C14.2, C15.2, R17.2, R18.2, R20.2, U5.4 (GND), U5.6 (CLK), U5.8 (VCC), U6.4 (GND), U6.6 (CLK), U6.8 (VCC), U6.9 (EP), U7.15 (GND), U7.16 (GND), U7.17 (GND), U7.5 (FB), U7.6 (GND); no longer U3.3 (EN)
- net CS: now also R19.2, U5.1 (~{CS}), U6.1 (~{CS})
- net SCL: now also R14.2, R15.2
- net SCK/SCL renamed MOSI
- net MOSI: now also U6.5 (DI/IO_{0})
- net SDO/ADR renamed MISO
- net MISO: now also U5.2 (DO/IO_{1}), U6.2 (DO/IO_{1})
- new net: R16.1, R17.1, U5.7 (~{HOLD}/~{RESET}/IO_{3}), U6.7 (~{HOLD}/~{RESET}/IO_{3})
- new net: L1.1, U7.1 (SW), U7.2 (SW), U7.3 (SW)
- new net: R21.2, U7.4 (PG)
- new net: C14.1, U7.9 (SS/TR)
- new net: R18.1, R19.1, R20.1, U5.3 (~{WP}/IO_{2}), U5.5 (DI/IO_{0}), U6.3 (~{WP}/IO_{2})
- new net: R14.1, R15.1
- new net AVID: U7.10 (VIN), U7.11 (VIN), U7.12 (VIN), U7.13 (EN)
- new net FSW: C15.1, L1.2, R21.1, U7.14 (VOS)
- new net IO3/Hold: R16.2
Other:
- note added: "+"
- note added: "-"
- note added: "Connectors"
- note added: "Jumpers"
- note added: "NOR Flash"
- note added: "Power 模組"
- note added: "QWIC_RIGHT_ANGLE"
- note added: "TP1"
- note added: "TP2"
- note added: "TP3"
- note added: "TP5"
- note added: "Testpoint"
- note added: "cut trace to disconnect Power LED"
- note added: "cut trace to remove I2C pull-up resistors"
- note added: "lout"
- moved on the sheet: C10, C11, D3, R12, R13, U1
