File: SmallAvionic/Ray/Ray.kicad_sch (KiCad schematic)
At the start: 52 parts, among them Q1 NMOS, Q2 NMOS, Q3 BSS138, Q4 BSS138, U1 STM32F103C8Tx, U2 BMI088, U3 AP2112K-3.3, U4 XC6206PxxxMR, U5 W25Q128JVS, U6 W25Q128JVE, U7 TPS62142

Commit message: Ray finish Ground Station Schematic
Parts:
- added 10uF: C, symbol Device:C
- added 1uF: ~, symbol Device:C
- added 2.7K (x2): R, symbol Device:R
- added 3V3, Buck_5v, GND, V_BAT+: TestPoint, symbol Connector:TestPoint
- added C16: 10p, symbol Device:C
- added C16, C27: 10u, symbol Device:C
- added C17, C18, C19, C21 (x2), C23 (x2), C25, C26: 100n, symbol Device:C
- added C17, C18, C19, C22, C24: 47u, symbol Device:C
- added C20, C22, C24: 4.7u, symbol Device:C
- added C28: 1n, symbol Device:C
- added C29, C30: 22pF, symbol Device:C
- added C31, C32, C33, C34: 100nF, symbol Device:C
- added D4: TVS, symbol Device:D_TVS_Filled
- added D5: G_5V, symbol Device:LED
- added D6: B_3V3, symbol Device:LED
- added F1: Fuse, symbol Device:Fuse
- added FB1: FerriteBead 120R @ 100M, symbol Device:FerriteBead
- added I2C_PU0: S_MODE, SparkFun_Magnetometer_MMC5983MA_Qwiic_Micro:SMT-JUMPER_3_2-NC_TRACE_SILK, symbol SparkFun_Magnetometer_MMC5983MA_Qwiic_Micro-eagle-import:JUMPER-SMT_3_2-NC_TRAC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
- added J1: Boot_mode_pin, symbol Connector:Conn_01x02_Pin
- added J2: USB_C_Receptacle_USB2.0_16P, symbol Connector:USB_C_Receptacle_USB2.0_16P
- added J3: Conn_01x04, symbol Connector_Generic:Conn_01x04
- added J5: Conn_01x02, symbol Connector_Generic:Conn_01x02
- added L2: 6.8u, symbol Device:L
- added LED0: JUMPER-SMT_2_NC_TRACE_SILK, SparkFun_Magnetometer_MMC5983MA_Qwiic_Micro:SMT-JUMPER_2_NC_TRACE_SILK, symbol SparkFun_Magnetometer_MMC5983MA_Qwiic_Micro-eagle-import:JUMPER-SMT_2_NC_TRACE_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
- added Q5, Q6: TSM3481CX6 RFG, Package_TO_SOT_SMD:SOT-23, symbol Transistor_FET:IRLML6402
- added R16(PG_pull_up), R28, R30, R34: 100k, symbol Device:R
- added R22, R23, R26, R27: 10k, symbol Device:R
- added R24, R25, R36, R37: 22ohm, symbol Device:R
- added R29: 18k, symbol Device:R
- added R31: 220k, symbol Device:R
- added R32: 1M, symbol Device:R
- added R33: 30k, symbol Device:R
- added R35: 0 ohm, symbol Device:R
- added R38, R39: 1k, symbol Device:R
- added R40: 1.5k, symbol Device:R
- added R41, R42: 5.1k, symbol Device:R
- added SW1: SW_Push, symbol Switch:SW_Push
- added U1: LD1117S33TR_SOT223, Package_TO_SOT_SMD:SOT-223-3_TabPin2, symbol Regulator_Linear:LD1117S33TR_SOT223
- added U10: TPS54538RQFR, VQFN-HR9_RQF_TEX, symbol Small_av_tony_lib:TPS54538RQFR
- added U11, U13: BMI088, Package_LGA:Bosch_LGA-16_4.5x3mm_P0.5mm_LayoutBorder7x1y_ClockwisePinNumbering, symbol Sensor_Motion:BMI088
- added U12: STM32F103C8Tx, Package_QFP:LQFP-48_7x7mm_P0.5mm, symbol MCU_ST_STM32F1:STM32F103C8Tx
- added U8: STM32F405VGTx, Package_QFP:LQFP-100_14x14mm_P0.5mm, symbol MCU_ST_STM32F4:STM32F405VGTx
- added U9: LTC4412xS6, Package_TO_SOT_SMD:TSOT-23-6, symbol Power_Management:LTC4412xS6
- added UMMC5983MA: ~, symbol MMC5983ma_Ray:MMC5983ma
- added Y1: 8Mhz, symbol Device:Crystal_GND24
Connections:
- net 3v3: now also U1.23 (VSS), U1.35 (VSS), U1.47 (VSS), U1.8 (VSSA), 10uF.1, 1uF.2, C16.2, C17.2, C17.2, C18.2, C18.2, C19.2, C19.2, C20.2, C21.2, C21.2, C22.2, C22.2, C23.2, C23.2, C24.2, C24.2, C25.2, C26.2, C27.2, C28.2, C29.2, C30.2, C31.1, C31.2, C32.1, C32.2, C33.1, C33.2, C34.1, C34.2, D4.1 (A1), D5.1 (K), D6.1 (K), GND.1, I2C_PU0.2, J2.A1 (GND), J2.A12 (GND), J2.B1 (GND), J2.B12 (GND), J2.S1 (SHIELD), J3.4 (Pin_4), J5.2 (Pin_2), LED0.1, R22.2, R23.2, R27.2, R28.2, R29.2, R32.2, R33.2, R41.2, R42.2, SW1.1, U1.1 (GND), U10.4 (GND), U13.11 (VDDIO), U13.2 (GNDA), U13.3 (VDD), U13.4 (GNDA), U13.6 (GNDIO), U13.7 (PS), U9.2 (GND), UMMC5983MA.5 (SDO), Y1.2 (G), Y1.4 (G); no longer D3.1 (K)
- net MISO: now also U13.10 (SDO2), U13.15 (SDO1)
- net MOSI: now also U13.9 (SDI/SDA)
- net at R14.1: now also I2C_PU0.1; no longer R15.1
- net +3.3V: now reaches U1.1 (VBAT)
- net +3.3V: now also U1.24 (VDD), U1.36 (VDD), U1.48 (VDD), 3V3.1, C16.1, C17.1, C18.1, C21.1, C21.1, C22.1, C23.1, C24.1, J1.1 (Pin_1), J3.1 (Pin_1), R26.1, R34.1, R39.2, R40.2, U1.2 (VO)
- net BOOT1: now reaches U1.20 (PB2)
- net BOOT1: now also R22.1
- net USB_D-: now reaches U1.32 (PA11)
- net USB_D-: now also R36.2
- net USB_D+: now reaches U1.33 (PA12)
- net USB_D+: now also R37.1, R40.1
- net SWDIO: now reaches U1.34 (PA13)
- net SWDIO: now also R24.1
- net SWCLK: now reaches U1.37 (PA14)
- net SWCLK: now also R25.1
- net BOOT0: now reaches U1.44 (BOOT0)
- net BOOT0: now also J1.2 (Pin_2), R23.1
- net HSE_IN: now reaches U1.5 (PD0)
- net HSE_IN: now also C29.1, Y1.1
- net HSE_OUT: now reaches U1.6 (PD1)
- net HSE_OUT: now also R35.1, Y1.3
- net RST: now reaches U1.7 (NRST)
- net RST: now also C19.1, SW1.2
- net +3.3VA: now reaches U1.9 (VDDA)
- net +3.3VA: now also C26.1, C27.1, FB1.1
- net SCK_3V renamed SCK
- net SCK: now also U13.8 (SCK/SCL)
- new net: C16.2, R31.2, R33.1, U10.3 (FB)
- new net: D6.2 (A), R39.1
- new net: Q6.1 (G), U9.5 (GATE)
- new net: J3.3 (Pin_3), R25.2, R27.1
- new net: R29.1, U10.7 (MODE)
- new net: L2.2, U10.8 (SW)
- new net: F1.1, J5.1 (Pin_1)
- new net: D4.2 (A2), F1.2, Q5.3 (D)
- new net: 10uF.2, UMMC5983MA.5 (SDO)
- new net: J2.A5 (CC1), R41.1
- new net: J2.A6 (D+), J2.B6 (D+), R37.2
- new net: J2.A7 (D-), J2.B7 (D-), R36.1
- new net: J2.B5 (CC2), R42.1
- new net: J3.2 (Pin_2), R24.2, R26.2
- new net: R30.1, R32.1, U9.3 (CTL)
- new net: D3.1 (K), LED0.2
- new net: U11.2 (GNDA), U11.4 (GNDA)
- new net: C28.1, FB1.2
- new net: I2C_PU0.3, R15.1
- new net: D5.2 (A), R38.1
- new net: C30.1, R35.2
- new net: U8.10 (VSS), U8.27 (VSS), U8.74 (VSS), U8.99 (VSS)
- new net: U12.23 (VSS), U12.35 (VSS), U12.47 (VSS)
- new net: Q5.1 (G), R28.1
- new net +USB_5V: J2.A4 (VBUS), J2.A9 (VBUS), J2.B4 (VBUS), J2.B9 (VBUS), Q6.3 (D), R30.2, U9.6 (SENSE)
- new net BUCK_5V: Buck_5v.1, C16.1, C17.1, C18.1, C19.1, C23.1, L2.1, Q6.2 (S), R16(PG_pull_up).1, R31.1, R38.2, U1.3 (VI), U9.1 (VIN)
- new net CSB_ACCEL: U13.14 (~{CSB1}), U13.5 (~{CSB2})
- new net I2C1_SCL: 2.7K.1, U12.42 (PB6), UMMC5983MA.1 (SCL/SCK)
- new net I2C1_SDA: 2.7K.1, U12.43 (PB7), UMMC5983MA.5 (SDO)
- new net INT1_ACCEL: U13.16 (INT1)
- new net INT2_ACCEL: U13.1 (INT2)
- new net INT3_GYRO: U13.12 (INT3)
- new net INT4_GYRO: U13.13 (INT4)
- new net PG_BUCK: R16(PG_pull_up).2, U10.9 (SS/PG)
- new net POWER_2.8~3.6V: 1uF.1, UMMC5983MA.2 (NC)
- new net SPI1_MISO: U12.16 (PA6)
- new net SPI1_MOSI: U12.17 (PA7)
- new net SPI1_SCK: U12.15 (PA5)
- new net SUP_STAT: R34.2, U9.4 (STAT)
- new net VIO: 2.7K.2, 2.7K.2, UMMC5983MA.5 (SDO)
- new net V_BAT: U10.2 (EN)
- new net V_BAT+: C20.1, C22.1, C24.1, C25.1, Q5.2 (S), U10.5 (VIN), U10.6 (VIN), V_BAT+.1
- no-connect marks 2 -> 5
Other:
- note added: "Barometer - BMP390"
- note added: "Boot&Debug"
- note added: "Buck"
- note added: "External reset"
- note added: "HSE crystal"
- note added: "Indicator"
- note added: "LDO"
- note added: "MCU"
- note added: "Power"
- note added: "Reverse Protection"
- note added: "Serial Wire Debug"
- note added: "Test point"
- note added: "USB"
- note added: "decoupling"
