File: SmallAvionic/Tony/SmallAvionic.kicad_sch (KiCad schematic)
At the start: 68 parts, among them J1 Boot_mode_pin, J2 USB_C_Receptacle_USB2.0_16P, J3 Conn_01x04, J5 Conn_01x02, Q1 TSM3481CX6 RFG, Q2 TSM3481CX6 RFG, SW1 SW_Push, U1 STM32F103C8Tx, U2 LD1117S33TR_SOT223, U3 LTC4412xS6, U4 TPS54538RQFR, U5 BMI088, Y1 8Mhz

Commit message: complete small av,parachute board
Parts:
- added 5k, R22, R23, R26, R27, R28, R29, R40, R41: 10k, symbol Device:R
- added BZ1: Active Buzzer, symbol Device:Buzzer
- added C20, C25, C26, C27, C32, C35: 100n, symbol Device:C
- added C28, C30: 1u, symbol Device:C
- added C29: 10u, symbol Device:C
- added C31: 4.7u, symbol Device:C
- added D11: R, symbol Device:LED
- added D12: 1N4148, Diode_THT:D_DO-35_SOD27_P7.62mm_Horizontal, symbol Diode:1N4148
- added D8: G, symbol Device:LED
- added J10: Conn_01x04, symbol Connector_Generic:Conn_01x04
- added J4: Conn_01x03, symbol Connector_Generic:Conn_01x03
- added J6: Screw_Terminal_01x01, symbol Connector:Screw_Terminal_01x01
- added Q5: NMOS, symbol Simulation_SPICE:NMOS
- added R24, R25: 2.7k, symbol Device:R
- added R35, R38: 2.2k, symbol Device:R
- added R39: 1k, symbol Device:R
- added U6: BMP390, 10LGA_2X2X0p75_BOS, symbol Small_av_tony_lib:BMP390
- added U7: MMC5983MA, MMC5983MA_MEM, symbol Small_av_tony_lib:MMC5983MA
- added U8: W25Q128JVS, Package_SO:SOIC-8_5.3x5.3mm_P1.27mm, symbol Memory_Flash:W25Q128JVS
Connections:
- net +3.3VA is gone; now on net +3.3V: C6.1, C7.1, FB1.1, U1.9 (VDDA)
- net +3.3V: now also U5.11 (VDDIO), U5.3 (VDD), C20.1, C25.1, C26.1, C27.1, C28.1, C30.1, C31.1, C32.1, R22.2, R23.2, R24.1, R25.1, R26.2, R27.2, R28.1, R29.2, U6.1 (VDDIO), U6.10 (VDD), U7.13 (VDDIO), U7.2 (VDD), U7.4 (SPI_CS), U8.8 (VCC)
- net GND: now also U5.2 (GNDA), U5.4 (GNDA), U5.6 (GNDIO), U5.7 (PS), 5k.1, C20.2, C25.2, C26.2, C27.2, C28.2, C29.2, C30.2, C31.2, C32.2, C35.2, J10.3 (Pin_3), J10.4 (Pin_4), J4.3 (Pin_3), J6.1 (Pin_1), Q5.3 (S), R35.1, R38.1, R40.2, U6.3 (VSS), U6.8 (VSS), U6.9 (VSS), U7.11 (GND), U7.9 (GND), U8.4 (GND)
- net V_BAT+: now also BZ1.1 (+), D12.1 (K), R41.2
- net INT_Accel2: now reaches U5.1 (INT2)
- net INT_Accel2: now also U1.11 (PA1)
- net SPI1_MISO: now reaches U5.10 (SDO2)
- net SPI1_MISO: now also U1.16 (PA6), U5.15 (SDO1), U6.5 (SDO)
- net INT_Gyro: now reaches U5.12 (INT3)
- net INT_Gyro: now also U1.12 (PA2)
- net CSB_Accel: now reaches U5.14 (~{CSB1})
- net CSB_Accel: now also U1.14 (PA4), R22.1
- net INT_Accel1: now reaches U5.16 (INT1)
- net INT_Accel1: now also U1.10 (PA0)
- net CSB_Gyro: now reaches U5.5 (~{CSB2})
- net CSB_Gyro: now also U1.13 (PA3), R23.1
- net SPI1_SCK: now reaches U5.8 (SCK/SCL)
- net SPI1_SCK: now also U1.15 (PA5), U6.2 (SCK)
- net SPI1_MOSI: now reaches U5.9 (SDI/SDA)
- net SPI1_MOSI: now also U1.17 (PA7), U6.4 (SDI)
- net CSB_Baro: now reaches U1.18 (PB0)
- net CSB_Baro: now also R28.2, U6.6 (CSB)
- net Battery_Sensing: now reaches U1.19 (PB1)
- net Battery_Sensing: now also 5k.2, C35.1, R41.1
- net LED_SYS: now reaches U1.2 (PC13)
- net LED_SYS: now also D8.2 (A)
- net INT_Baro: now reaches U1.21 (PB10)
- net INT_Baro: now also U6.7 (INT)
- net Buzzer: now reaches U1.22 (PB11)
- net Buzzer: now also R39.2
- net WP_Flash: now reaches U1.25 (PB12)
- net WP_Flash: now also R27.1, U8.3 (~{WP}/IO_{2})
- net SPI2_SCK: now reaches U1.26 (PB13)
- net SPI2_SCK: now also U8.6 (CLK)
- net SPI2_MISO: now reaches U1.27 (PB14)
- net SPI2_MISO: now also U8.2 (DO/IO_{1})
- net SPI2_MOSI: now reaches U1.28 (PB15)
- net SPI2_MOSI: now also U8.5 (DI/IO_{0})
- net CSB_Flash: now reaches U1.29 (PA8)
- net CSB_Flash: now also R29.1, U8.1 (~{CS})
- net LED_State: now reaches U1.3 (PC14)
- net LED_State: now also D11.2 (A)
- net USART1_TX: now reaches U1.30 (PA9)
- net USART1_TX: now also J4.1 (Pin_1)
- net USART1_RX: now reaches U1.31 (PA10)
- net USART1_RX: now also J4.2 (Pin_2)
- net INT_Magn: now reaches U1.41 (PB5)
- net INT_Magn: now also U7.15 (INT)
- net I2C1_SCL: now reaches U1.42 (PB6)
- net I2C1_SCL: now also R24.2, U7.1 (SCL/SPI_SCK)
- net I2C1_SDA: now reaches U1.43 (PB7)
- net I2C1_SDA: now also R25.2, U7.16 (SDA/SPI_SDI)
- net FIRE: now reaches U1.45 (PB8)
- net FIRE: now also J10.2 (Pin_2)
- net PWM Servo: now reaches U1.46 (PB9)
- net PWM Servo: now also J10.1 (Pin_1)
- new net: R26.1, U8.7 (~{HOLD}/~{RESET}/IO_{3})
- new net: C29.1, U7.10 (CAP)
- new net: BZ1.2 (-), D12.2 (A), Q5.1 (D)
- new net: Q5.2 (G), R39.1, R40.1
- new net: D11.1 (K), R38.2
- new net: D8.1 (K), R35.2
- no-connect marks 3 -> 4
Other:
- added sheet Deployment Board (deployment_board.kicad_sch.kicad_sch)
- note added: "Barometer"
- note added: "Battery monitor"
- note added: "Connection to Main_AV"
- note added: "Flash"
- note added: "IMU"
- note added: "Ignition connector"
- note added: "Magnetometer"
- note added: "Power management"
- note added: "UART communication"
- note added: "common ground to Main_AV GND"
- note added: "decoupling for VDD,VDDIO"
- moved on the sheet: 3V3, Buck_5v, C12, C13, C14, C15, C16, C17, C18, C19, C21, C22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
