File: BigAvionic/_autosave-Iusbubula_Avionic_Board.kicad_sch (KiCad schematic)
At the start: 53 parts, among them J5 Conn_01x02, Q1 TSM3481CX6 RFG, Q2 TSM3481CX6 RFG, U1 STM32F405VGTx, U2 LD1117S33TR_SOT223, U3 LTC4412xS6, U4 TPS54538RQFR

Commit message: finished power of Big AV
Parts:
- added C20: 1n, symbol Device:C
Connections:
- net GND: now also C20.2
- net VREF: now reaches C11.1, C25.1, FB1.1, U1.22 (VDDA)
- net VREF: now also C20.1
Other:
- note added: "ESR<2ohm"
Changed lines of the file:
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@@
+		)
+	)
+	(text "ESR<2ohm\n"
+		(exclude_from_sim no)
+		(at 215.138 188.976 0)
+		(effects
+			(font
+				(size 1.27 1.27)
+			)
 		)
 	)
@@
 	)
 	(junction
+		(at 284.48 53.34)
+		(diameter 0)
+		(color 0 0 0 0)
+	)
+	(junction
 		(at 135.89 267.97)
 		(diameter 0)
@@
 	(junction
 		(at 201.93 39.37)
+		(diameter 0)
+		(color 0 0 0 0)
+	)
+	(junction
+		(at 273.05 39.37)
 		(diameter 0)
 		(color 0 0 0 0)
@@
 	(wire
 		(pts
-			(xy 266.7 39.37) (xy 284.48 39.37)
+			(xy 266.7 39.37) (xy 273.05 39.37)
 		)
 		(stroke
@@
 	(wire
 		(pts
+			(xy 273.05 49.53) (xy 273.05 53.34)
+		)
+		(stroke
+			(width 0)
+			(type default)
+		)
+	)
+	(wire
+		(pts
 			(xy 110.49 242.57) (xy 106.68 242.57)
 		)
@@
 	(wire
 		(pts
+			(xy 273.05 39.37) (xy 284.48 39.37)
+		)
+		(stroke
+			(width 0)
+			(type default)
+		)
+	)
+	(wire
+		(pts
 			(xy 115.57 346.71) (xy 115.57 359.41)
 		)
@@
 	(wire
 		(pts
+			(xy 273.05 39.37) (xy 273.05 41.91)
+		)
+		(stroke
+			(width 0)
+			(type default)
+		)
+	)
+	(wire
+		(pts
 			(xy 80.01 255.27) (xy 91.44 255.27)
 		)
@@
 		(pts
 			(xy 106.68 242.57) (xy 106.68 240.03)
+		)
+		(stroke
+			(width 0)
+			(type default)
+		)
+	)
+	(wire
+		(pts
+			(xy 273.05 53.34) (xy 284.48 53.34)
 		)
 		(stroke
@@
 		)
 	)
+	(global_label "VREF"
+		(shape input)
+		(at 266.7 39.37 90)
+		(fields_autoplaced yes)
+		(effects
+			(font
+				(size 1.27 1.27)
+			)
+			(justify left)
+		)
+		(property "Intersheetrefs" "${INTERSHEET_REFS}"
+			(at 266.7 31.7886 90)
+			(effects
+				(font
+					(size 1.27 1.27)
+				)
+				(justify left)
+				(hide yes)
+			)
+		)
+	)
 	(global_label "BUCK_5V"
 		(shape input)
@@
 		(property "Intersheetrefs" "${INTERSHEET_REFS}"
 			(at 102.87 289.5214 90)
+			(effects
+				(font
+					(size 1.27 1.27)
+				)
+				(justify right)
+				(hide yes)
+			)
+		)
+	)
+	(global_label "VREF"
+		(shape input)
+		(at 217.17 78.74 180)
+		(fields_autoplaced yes)
+		(effects
+			(font
+				(size 1.27 1.27)
+			)
+			(justify right)
+		)
+		(property "Intersheetrefs" "${INTERSHEET_REFS}"
+			(at 209.5886 78.74 0)
 			(effects
 				(font
@@
 					(unit 1)
 				)
+			)
+		)
+	)
+	(symbol
+		(lib_id "Device:C")
+		(at 273.05 45.72 0)
+		(unit 1)
+		(exclude_from_sim no)
+		(in_bom yes)
+		(on_board yes)
+		(dnp no)
+		(property "Reference" "C20"
+			(at 276.86 44.4499 0)
+			(effects
+				(font
+					(size 1.27 1.27)
+				)
+				(justify left)
+			)
+		)
+		(property "Value" "1n"
+			(at 276.86 46.9899 0)
+			(effects
+				(font
+					(size 1.27 1.27)
+				)
+				(justify left)
+			)
+		)
+		(property "Footprint" ""
+			(at 274.0152 49.53 0)
+			(effects
+				(font
+					(size 1.27 1.27)
+				)
+				(hide yes)
+			)
+		)
+		(property "Datasheet" "~"
+			(at 273.05 45.72 0)
+			(effects
+				(font
+					(size 1.27 1.27)
+				)
+				(hide yes)
+			)
+		)
+		(property "Description" "Unpolarized capacitor"
+			(at 273.05 45.72 0)
+			(effects
+				(font
+					(size 1.27 1.27)
+				)
+				(hide yes)
+			)
+		)
+		(pin "1"
+		)
+		(pin "2"
+		)
+		(instances
+			(project "Iusbubula_Avionic_Board"
+				(path "/80a059dc-2311-4dd3-afad-18a5367fc218"
+					(reference "C20")
+					(unit 1)
+				)
