File: BigAvionic/_autosave-Iusbubula_Avionic_Board.kicad_sch (KiCad schematic)
At the start: 104 parts, among them J1 Conn_01x02, J2 USB_C_Receptacle_USB2.0_16P, J3 Conn_01x04, J4 Conn_Coaxial, J5 Conn_01x02, Q1 TSM3481CX6 RFG, Q2 TSM3481CX6 RFG, SW1 SW_Push, U1 STM32F405VGTx, U2 LD1117S33TR_SOT223, U3 LTC4412xS6, U4 TPS54538RQFR, U5 BMI088, U6 BMP390, U7 MMC5983MA, U8 ADXL375BCCZ, U9 NEO-M9N-00B, Y1 8Mhz

Commit message: finish lora
Parts:
- added C43, C45: 100n, symbol Device:C
- added C44: 100u, symbol Device:C
- added C46: 22u, symbol Device:C
- added R30, R31: 22ohm, symbol Device:R
- added R32, R33: 10k, symbol Device:R
- added U10: E22-400T30S, symbol A_library:E22-XXXT30
- added U11: E80-900M23313S, symbol A_library:E80-xxxM2213S
Connections:
- net +3.3V: now also C43.1, C44.1, C45.1, C46.1, R32.2, R33.2, U10.2 (VCC), U11.25 (VCC)
- net GND: now also C43.2, C44.2, C45.2, C46.2, U10.1 (GND), U10.12 (GND), U10.13 (GND), U10.14 (GND), U10.23 (GND), U11.1 (GND), U11.19 (GND), U11.26 (GND), U11.8 (GND)
- net I2C1_SCL: now also U1.93 (PB7); no longer U1.92 (PB6)
- net I2C1_SDA: now also U1.95 (PB8); no longer U1.93 (PB7)
- net INT_Magn: now also U1.92 (PB6); no longer U1.91 (PB5)
- net UART6_RX: now also R11.1; no longer R12.1
- net UART6_TX: now also R12.1; no longer R11.1
- net UART3_TX: now reaches U1.55 (PD8)
- net UART3_TX: now also R30.2
- net UART3_RX: now reaches U1.56 (PD9)
- net UART3_RX: now also R31.2
- net LORA433_M1: now reaches U1.57 (PD10)
- net LORA433_M1: now also U10.6 (M1)
- net LORA433_M0: now reaches U1.58 (PD11)
- net LORA433_M0: now also U10.7 (M0)
- net LORA433_RST: now reaches U1.59 (PD12)
- net LORA433_RST: now also R32.1, U10.22 (RESET)
- net LORA920_INT: now reaches U1.85 (PD4)
- net LORA920_INT: now also U11.22 (DIO9)
- net LORA920_RST: now reaches U1.86 (PD5)
- net LORA920_RST: now also R33.1, U11.21 (LR_NRST)
- net LORA920_BUSY: now reaches U1.87 (PD6)
- net LORA920_BUSY: now also U11.7 (BUSY)
- net CSB_LORA920: now reaches U1.88 (PD7)
- net CSB_LORA920: now also U11.6 (NSS)
- net SPI3_SCK: now reaches U1.89 (PB3)
- net SPI3_SCK: now also U11.5 (SCK)
- net SPI3_MISO: now reaches U1.90 (PB4)
- net SPI3_MISO: now also U11.3 (MISO)
- new net: R31.1, U10.4 (TXD)
- new net: R30.1, U10.5 (RXD)
- new net LORA433_BUSY: U10.3 (AUX)
- new net SPI3_MOSI: U1.91 (PB5), U11.4 (MOSI)
- no-connect marks 18 -> 26
Other:
- note added: "LORA 433"
- note added: "LORA 920"
- note added: "using ipx in the lora model"

Commit message: finish sd
Parts:
- added C47: 10u, symbol Device:C
- added C48: 100n, symbol Device:C
- added J6: Micro_SD_Card_Det1, symbol Connector:Micro_SD_Card_Det1
- added R34, R36, R37, R39, R42, R43: 22ohm, symbol Device:R
- added R35, R38, R40, R41, R44: 47k, symbol Device:R
Connections:
- net +3.3V: now also C47.1, C48.1, J6.4 (VDD), R35.2, R38.2, R40.2, R41.2, R44.2
- net GND: now also C47.2, C48.2, J6.10 (SHIELD), J6.6 (VSS)
- net SDIO_D0: now reaches U1.65 (PC8)
- net SDIO_D0: now also R42.2
- net SDIO_D1: now reaches U1.66 (PC9)
- net SDIO_D1: now also R43.2
- net SDIO_D2: now reaches U1.78 (PC10)
- net SDIO_D2: now also R34.2
- net SDIO_D3: now reaches U1.79 (PC11)
- net SDIO_D3: now also R36.2
- net SDIO_CK: now reaches U1.80 (PC12)
- net SDIO_CK: now also R37.2, R39.2
- net SDIO_CMD: now reaches U1.83 (PD2)
- net SDIO_DET: now reaches U1.84 (PD3)
- net SDIO_DET: now also J6.9 (DET)
- new net: J6.3 (CMD), R39.1, R40.1
- new net: J6.7 (DAT0), J6.8 (DAT1), R41.1, R42.1, R43.1, R44.1
- new net: J6.5 (CLK), R37.1
- new net: J6.2 (DAT3/CD), R36.1, R38.1
- new net: J6.1 (DAT2), R34.1, R35.1
Other:
- note added: "SD card"
