File: BigAvionic/_autosave-Iusbubula_Avionic_Board.kicad_sch (KiCad schematic)
At the start: 156 parts, among them J1 Conn_01x02, J10 Conn_01x04, J12 Conn_01x04, J2 USB_C_Receptacle_USB2.0_16P, J3 Conn_01x04, J4 Conn_Coaxial, J5 Conn_01x02, J6 Micro_SD_Card_Det1, J7 Screw_Terminal_01x01, J8 Conn_01x03, Q1 TSM3481CX6 RFG, Q2 TSM3481CX6 RFG, Q5 NMOS, SW1 SW_Push, SW2 USER_Buttom, SW3 USER_Buttom, U1 STM32F405VGTx, U10 E22-400T30S, U11 E80-900M23313S, U12 W25Q128JVS, U2 LD1117S33TR_SOT223, U3 LTC4412xS6, U4 TPS54538RQFR, U5 BMI088, U6 BMP390, U7 MMC5983MA, U8 ADXL375BCCZ, U9 NEO-M9N-00B, Y1 8Mhz

Commit message: 3/4
Parts:
- removed 5k: 10k, symbol Device:R
- removed J8: Conn_01x03, symbol Connector_Generic:Conn_01x03
- removed R5: 0ohm, symbol Device:R
- added J9: Conn_01x04, Connector_JST:JST_EH_S4B-EH_1x04_P2.50mm_Horizontal, symbol Connector_Generic:Conn_01x04
- added R54: 0ohm, symbol Device:R
- added R55: 5k, symbol Device:R
- 3V3: footprint (none) -> TestPoint:TestPoint_Pad_D1.0mm
- BZ1: footprint (none) -> Buzzer_Beeper:Buzzer_12x9.5RM7.6
- Buck_5v1: renamed from Buck_5v; footprint (none) -> TestPoint:TestPoint_Pad_D1.0mm
- C1, C10, C11, C12, C13, C14, C15, C16, C17, C18, C19, C2, C20, C21, C22, C23, C24, C25, C26, C27, C28, C29, C3, C30, C31, C32, C33, C34, C35, C36, C37, C38, C39, C4, C40, C41, C42, C43, C44, C45, C46, C47, C48, C49, C5, C50, C51, C52, C53, C6, C7, C8, C9: footprint (none) -> Capacitor_SMD:C_0805_2012Metric_Pad1.18x1.45mm_HandSolder
- D1, D11, D2, D3, D4, D5, D8: footprint (none) -> LED_SMD:LED_0805_2012Metric_Pad1.15x1.40mm_HandSolder
- D12: footprint Diode_THT:D_DO-35_SOD27_P7.62mm_Horizontal -> LED_SMD:LED_0805_2012Metric_Pad1.15x1.40mm_HandSolder
- F1: footprint (none) -> Fuse:Fuse_0805_2012Metric_Pad1.15x1.40mm_HandSolder
- FB1: footprint (none) -> Inductor_SMD:L_0805_2012Metric_Pad1.05x1.20mm_HandSolder
- GND1: renamed from GND; footprint (none) -> TestPoint:TestPoint_Pad_1.0x1.0mm
- J1: footprint (none) -> Connector_PinHeader_2.54mm:PinHeader_1x02_P2.54mm_Vertical
- J10: footprint (none) -> Connector_JST:JST_EH_S4B-EH_1x04_P2.50mm_Horizontal
- J12: footprint (none) -> Connector_JST:JST_EH_B4B-EH-A_1x04_P2.50mm_Vertical
- J2: footprint (none) -> Connector_USB:USB_C_Receptacle_HRO_TYPE-C-31-M-12
- J3: footprint (none) -> Connector_PinHeader_2.54mm:PinHeader_1x04_P2.54mm_Vertical
- J4: footprint (none) -> Connector_Coaxial:U.FL_Hirose_U.FL-R-SMT-1_Vertical
- J5: footprint (none) -> Connector_JST:JST_PH_S2B-PH-K_1x02_P2.00mm_Horizontal
- J6: footprint (none) -> Connector_Card:microSD_HC_Molex_47219-2001
- J7: footprint (none) -> TerminalBlock_Phoenix:TerminalBlock_Phoenix_PT-1,5-2-3.5-H_1x02_P3.50mm_Horizontal
- renumbered R16(PG_pull_up) to R16(PG_pull_up)1, V_BAT+ to V_BAT+1
Connections:
- net Battery_Sensing: now also R55.2
- net GND: now also J9.3 (Pin_3), R55.1
- net USART2_RX: now also J9.1 (Pin_1)
- net USART2_TX: now also J9.2 (Pin_2)
- net USB_D+: now also R54.2
- net at J2.A6 (D+), J2.B6 (D+): now also R54.1
- net RST renamed RESET
- net RESET: now also J9.4 (Pin_4)
- no-connect marks 26 -> 46
