File: BigAvionic/Iusbubula_Avionic_Board.kicad_sch (KiCad schematic)
At the start: 154 parts, among them J1 Conn_01x02, J10 Conn_01x04, J12 Conn_01x04, J2 USB_C_Receptacle_USB2.0_16P, J3 Conn_01x04, J4 Conn_Coaxial, J5 Conn_01x02, J6 Micro_SD_Card_Det1, J7 Screw_Terminal_01x01, J9 Conn_01x04, Q1 TSM3481CX6 RFG, Q2 TSM3481CX6 RFG, Q5 NMOS, SW1 SW_Push, SW2 USER_Buttom, SW3 USER_Buttom, U1 STM32F405VGTx, U10 E22-400T30S, U11 E80-900M23313S, U12 W25Q128JVS, U2 LD1117S33TR_SOT223, U3 LTC4412xS6, U4 TPS54538RQFR, U5 BMI088, U6 BMP390, U7 MMC5983MA, U8 ADXL375BCCZ, U9 NEO-M9N-00B, Y1 8Mhz

Commit message: jpush
Parts:
- added L2: short, symbol Device:L
- added R27: NC, symbol Device:R
- L1: footprint Inductor_SMD:L_7.3x7.3_H3.5 -> (none)
- Q5: footprint Package_TO_SOT_SMD:SOT-23 -> (none)
- R1, R10, R11, R12, R13, R14, R15, R16, R16(PG_pull_up)1, R17, R18, R19, R2, R20, R21, R22, R23, R24, R25, R26, R28, R29, R3, R30, R31, R32, R33, R34, R35, R36, R37, R38, R39, R4, R40, R41, R42, R43, R44, R45, R46, R47, R48, R49, R5, R50, R51, R52, R53, R54, R55, R6, R7, R8, R9: footprint Resistor_SMD:R_0805_2012Metric_Pad1.20x1.40mm_HandSolder -> (none)
- SW1, SW2, SW3: footprint Button_Switch_THT:SW_PUSH_6mm_H4.3mm -> (none)
- TP1, V_BAT+1: footprint TestPoint:TestPoint_Pad_D1.0mm -> (none)
- U9: footprint Tony:SMT_9N-00B_UBL -> (none)
- Y1: footprint Crystal:Crystal_HC49-U_Vertical -> (none)
Connections:
- net at C41.1, C42.1: now also L2.2, R27.1; no longer J4.1 (In)
- net at U9.9 (VCC_RF): now also R27.2
- new net: J4.1 (In), L2.1
- no-connect marks 47 -> 46
Other:
- note added: "Reserved for active atenna"
- moved on the sheet: C41
