File: BigAvionic/Iusbubula_Avionic_Board.kicad_sch (KiCad schematic)
At the start: 154 parts, among them J1 Conn_01x02, J10 Conn_01x04, J12 Conn_01x04, J2 USB_C_Receptacle_USB2.0_16P, J3 Conn_01x04, J4 Conn_Coaxial, J5 Conn_01x02, J6 Micro_SD_Card_Det1, J7 Screw_Terminal_01x01, J9 Conn_01x04, Q1 TSM3481CX6 RFG, Q2 TSM3481CX6 RFG, Q5 NMOS, SW1 SW_Push, SW2 USER_Buttom, SW3 USER_Buttom, U1 STM32F405VGTx, U10 E22-400T30S, U11 E80-900M23313S, U12 W25Q128JVS, U2 LD1117S33TR_SOT223, U3 LTC4412xS6, U4 TPS54538RQFR, U5 BMI088, U6 BMP390, U7 MMC5983MA, U8 ADXL375BCCZ, U9 NEO-M9N-00B, Y1 8Mhz

Commit message: tony
Parts:
- U10: footprint (none) -> Tony:XCVR_E22-900T30S
- U11: footprint (none) -> Tony:E80-xxxM2213S
- U4: footprint (none) -> Tony:VQFN-HR9_RQF_TEX(TPS54538)
- U6: footprint (none) -> Tony:10LGA_2X2X0p75_BOS-M
- U7: footprint (none) -> Tony:MMC5983MA_MEM
- U8: footprint (none) -> Tony:LGA_CC-14-1_ADI-L
Other:
- added sheet top layer (untitled.kicad_sch)
Changed lines of the file:
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@@
 			)
 		)
-		(property "Footprint" ""
+		(property "Footprint" "Tony:10LGA_2X2X0p75_BOS-M"
 			(at 260.35 106.68 0)
 			(effects
@@
 			)
 		)
-		(property "Footprint" ""
+		(property "Footprint" "Tony:LGA_CC-14-1_ADI-L"
 			(at 251.46 40.64 0)
 			(effects
@@
 			)
 		)
-		(property "Footprint" ""
+		(property "Footprint" "Tony:VQFN-HR9_RQF_TEX(TPS54538)"
 			(at 161.29 250.19 0)
 			(effects
@@
 			)
 		)
-		(property "Footprint" ""
+		(property "Footprint" "Tony:XCVR_E22-900T30S"
 			(at 397.51 180.34 0)
 			(effects
@@
 			)
 		)
-		(property "Footprint" ""
+		(property "Footprint" "Tony:MMC5983MA_MEM"
 			(at 378.46 39.37 0)
 			(effects
@@
 			)
 		)
-		(property "Footprint" ""
+		(property "Footprint" "Tony:E80-xxxM2213S"
 			(at 488.95 187.96 0)
 			(effects
@@
 				)
 			)
+		)
+	)
+	(sheet
+		(at 505.46 46.99)
+		(size 73.66 69.85)
+		(exclude_from_sim no)
+		(in_bom yes)
+		(on_board yes)
+		(dnp no)
+		(fields_autoplaced yes)
+		(stroke
+			(width 0.1524)
+			(type solid)
+		)
+		(fill
+			(color 0 0 0 0.0000)
+		)
+		(property "Sheetname" "top layer"
+			(at 505.46 46.2784 0)
+			(effects
+				(font
+					(size 1.27 1.27)
+				)
+				(justify left bottom)
+			)
+		)
+		(property "Sheetfile" "untitled.kicad_sch"
+			(at 505.46 117.4246 0)
+			(effects
+				(font
+					(size 1.27 1.27)
+				)
+				(justify left top)
+			)
+		)
+		(instances
+			(project "Iusbubula_Avionic_Board"
+				(path "/80a059dc-2311-4dd3-afad-18a5367fc218"
+					(page "2")
+				)
+			)
