File: GroundStation/GroundStation/GroundStation.kicad_pcb (KiCad board)
At the start: 2 copper layers, 70 parts, among them J1 SD_Card_Receptacle, J4 Conn_Coaxial, J5 Conn_01x02, P1 USB_C_Plug_USB2.0, Q1 TSM3481CX6 RFG, U1 STM32F103C8Tx, U101 LD1117S33TR_SOT223, U2 E22-400T30S_LoRa, U4 TPS54538RQFR, U9 NEO-M9N-00B

Commit message: jpush
Routing:
- net GND: track 0.00 -> 551.6 mm, vias 0 -> 8
- net 3.3V: track 0.00 -> 210.8 mm, vias 0 -> 2
- net BUCK_5V: track 0.00 -> 168.7 mm, vias 0 -> 4
- net V_BAT+: track 0.00 -> 159.7 mm, vias 0 -> 2
- net +3.3V: track 0.00 -> 119.1 mm
- net Net-(U9-SAFEBOOT_N): track 0.00 -> 77.5 mm
- net Net-(J4-In): track 0.00 -> 59.8 mm
- net USART1_GPS_RESET: track 0.00 -> 53.8 mm, vias 0 -> 2
- net USART2_LoRa1_NRST: track 0.00 -> 47.1 mm
- net Net-(U1-VDDA): track 0.00 -> 44.1 mm, vias 0 -> 3
- net Net-(D102-A1): track 0.00 -> 32.7 mm, vias 0 -> 2
- net Net-(C41-Pad1): track 0.00 -> 30.2 mm, vias 0 -> 2
- net SPI2_SDcard_CS: track 0.00 -> 28.4 mm
- net USART1_GPS_TX: track 0.00 -> 26.2 mm, vias 0 -> 2
- net SPI2_SDcard_SCK: track 0.00 -> 25.7 mm
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