File: GroundStation/GroundStation/GroundStation.kicad_pcb (KiCad board)
At the start: 4 copper layers, 83 x 108.3 mm, 72 parts, among them J1 SD_Card_Receptacle, J4 Conn_Coaxial, J5 Conn_01x02, P1 USB_C_Plug_USB2.0, Q1 TSM3481CX6 RFG, U1 STM32F103C8Tx, U10 E22-400T30S, U101 LD1117S33TR_SOT223, U11 E80-900M23313S, U4 TPS54538RQFR, U9 NEO-M9N-00B

Commit message: test
Parts:
- moved Buck_5v101 50.4 mm to (107.9, 101.7)
- moved D101 38.2 mm to (115.2, 101.8)
- moved R16 38.2 mm to (115.1, 104.3)
Routing:
- net GND: track 329.1 -> 378.5 mm, vias 23 -> 28
- net +3.3V: track 33.2 -> 58.0 mm, vias 6 -> 10
- net BUCK_5V: track 117.5 -> 133.9 mm
- net USART2_LoRa1_NRST: track 52.1 -> 60.7 mm
- net Net-(D101-A): track 0.00 -> 2.57 mm
- net Net-(D2-A): track 0.00 -> 2.54 mm
- net USART2_LoRa1_AUX: track 60.4 -> 62.0 mm
- net SPI2_SDcard_MOSI: track 42.4 -> 43.6 mm
- net USART2_LoRa1_M0: track 58.6 -> 59.7 mm
- net SPI1_LoRa2_SCK: track 44.5 -> 45.3 mm
- net USART1_GPS_TX: track 31.6 -> 31.5 mm, vias 4 -> 3
- net Net-(U9-SAFEBOOT_N): vias 3 -> 2
- net (no net): vias 1 -> 0
