File: BigAvionic/top layer/top_layer.kicad_sch (KiCad schematic)
At the start: 19 parts, among them J4 Conn_Coaxial, J8 Conn_01x02, U7 MMC5983MA, U9 NEO-M9N-00B

Commit message: finish first layer of big av
Parts:
- removed C41: NC, Capacitor_SMD:C_0805_2012Metric_Pad1.18x1.45mm_HandSolder, symbol Device:C
- removed C42: 100p, Capacitor_SMD:C_0805_2012Metric_Pad1.18x1.45mm_HandSolder, symbol Device:C
- removed J8: Conn_01x02, symbol Connector_Generic:Conn_01x02
- removed R11: 22ohm, Resistor_SMD:R_0805_2012Metric_Pad1.20x1.40mm_HandSolder, symbol Device:R
- added C8: 100n, Capacitor_SMD:C_0805_2012Metric_Pad1.18x1.45mm_HandSolder, symbol Device:C
- added C9: 10u, Capacitor_SMD:C_0805_2012Metric_Pad1.18x1.45mm_HandSolder, symbol Device:C
- added J1: Conn_01x08, Connector_JST:JST_GH_SM08B-GHS-TB_1x08-1MP_P1.25mm_Horizontal, symbol Connector_Generic:Conn_01x08
- added J3: Conn_01x04, Connector_JST:JST_GH_SM04B-GHS-TB_1x04-1MP_P1.25mm_Horizontal, symbol Connector_Generic:Conn_01x04
- renumbered C33 to C1, C34 to C4, C35 to C5, C39 to C6, C40 to C7, D4 to D1, J4 to J2, R26 to R1, R29 to R2, R24 to R3, R25 to R4, R12 to R5, U9 to U1, U7 to U2
Connections:
- net +3.3V: now also C8.1, C9.1, J3.1 (Pin_1), J3.2 (Pin_2)
- net GND: now also C8.2, C9.2, J1.3 (Pin_3), J1.6 (Pin_6), J3.3 (Pin_3), J3.4 (Pin_4)
- net I2C1_SCL: now also J1.5 (Pin_5)
- net I2C1_SDA: now also J1.4 (Pin_4)
- net INT_Magn: now also J1.7 (Pin_7)
- net RST_GPS: now also J1.8 (Pin_8)
- net UART6_RX: now also U1.20 (TXD_/_SPI_MISO), J1.2 (Pin_2)
- net UART6_TX: now also J1.1 (Pin_1)
- net at J2.1 (In): now also U1.11 (RF_IN)

Commit message: save
Parts:
- added H1, H2, H3, H4: MountingHole, MountingHole:MountingHole_3.2mm_M3_DIN965_Pad, symbol Mechanical:MountingHole
