File: Deployment board/Deployment board.kicad_sch (KiCad schematic)
At the start: 32 parts, among them J1 Conn_01x03, J2 Conn_01x03, J3 Conn_01x02, J4 Conn_01x02, J5 Conn_01x02, J6 XT60, J7 Conn_01x02, Q1 IRLR7843, Q2 IRLR7843, Q3 FDD4141, Q4 IRLR7843

Commit message: jpush
Parts:
- J5: footprint Connector_JST:JST_EH_B2B-EH-A_1x02_P2.50mm_Vertical -> Connector_Molex:Molex_Micro-Fit_3.0_43650-0221_1x02_P3.00mm_Vertical
Changed lines of the file:
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@@
 			)
 		)
-		(property "Footprint" "Connector_JST:JST_EH_B2B-EH-A_1x02_P2.50mm_Vertical"
+		(property "Footprint" "Connector_Molex:Molex_Micro-Fit_3.0_43650-0221_1x02_P3.00mm_Vertical"
 			(at 130.81 30.48 0)
 			(effects
