File: Deployment board/Deployment board.kicad_sch (KiCad schematic)
At the start: 52 parts, among them J1 Conn_01x02, J2 Conn_01x02, J3 Conn_01x02, J4 Conn_01x04, J5 Conn_01x04, J6 Conn_01x02, J7 Conn_01x02, M1 Motor_Servo, M2 Motor_Servo, Q1 IRLR7843, Q2 IRLR7843, Q3 FDD4141, U1 TPSM84824MOLR

Commit message: deployment board
Parts:
- R10, R11: value 3.3k -> ~
Changed lines of the file:
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@@
 			)
 		)
-		(property "Value" "3.3k"
+		(property "Value" "~"
 			(at 179.578 89.662 90)
 			(effects
@@
 			)
 		)
-		(property "Value" "3.3k"
+		(property "Value" "~"
 			(at 178.308 68.072 90)
 			(effects

Commit message: deployment board
Parts:
- removed C6: 1000u, Capacitor_SMD:CP_Elec_10x14.3, symbol Device:C_Polarized
- removed C7, C8: 10uF 3.979mOhm, Capacitor_SMD:C_0805_2012Metric_Pad1.18x1.45mm_HandSolder, symbol Device:C
- removed C9: 47uF 2.674mOhm Qty=3, Capacitor_SMD:C_0805_2012Metric_Pad1.18x1.45mm_HandSolder, symbol Device:C
- removed D2, D4: D_Schottky, Diode_SMD:D_SMA-SMB_Universal_Handsoldering, symbol Device:D_Schottky
- removed D7: Indicater, LED_SMD:LED_1206_3216Metric_Pad1.42x1.75mm_HandSolder, symbol Device:LED
- removed Q3: FDD4141, Package_TO_SOT_SMD:SOT-23, symbol Transistor_FET:IRLML6402
- removed R12: 10k, Resistor_SMD:R_0805_2012Metric_Pad1.20x1.40mm_HandSolder, symbol Device:R
- removed R13: 866k, Resistor_SMD:R_0805_2012Metric_Pad1.20x1.40mm_HandSolder, symbol Device:R
- removed R14: 6.81k, Resistor_SMD:R_0805_2012Metric_Pad1.20x1.40mm_HandSolder, symbol Device:R
- removed R15: 34.8k, Resistor_SMD:R_0805_2012Metric_Pad1.20x1.40mm_HandSolder, symbol Device:R
- removed R2, R7: 1k, Resistor_SMD:R_0805_2012Metric_Pad1.20x1.40mm_HandSolder, symbol Device:R
- removed U1: TPSM84824MOLR, TPSM84824:MOL0024A, symbol TPSM84824:TPSM84824MOLR
- added C7, C8, C9: 220uF,865060657012, Capacitor_SMD:CP_Elec_10x10.5, symbol Device:C_Polarized
- added D12, D7, D8: D_Schottky,PMEG3030EP,115, Diode_SMD:D_SOD-128, symbol Device:D_Schottky
- added D5: LED,AP3216ID, LED_SMD:LED_1206_3216Metric_Pad1.42x1.75mm_HandSolder, symbol Device:LED
- added L1: 33uH,SRN3010BTA-330M, Inductor_SMD_Wurth:L_Wurth_WE-LQSH-3012, symbol Device:L
- added Q3: SI7613DN-T1-GE3, Package_SO:Vishay_PowerPAK_1212-8_Single, symbol Transistor_FET:SiS415DNT
- added U1: LM2596S-5.0/NOPB, Package_TO_SOT_SMD:TO-263-5_TabPin3, symbol 2026-05-01_10-47-38:LM2596S-12_NOPB
- C1, C2, C5: value 1000u -> 220uF,865060657012; footprint Capacitor_SMD:CP_Elec_10x14.3 -> Capacitor_SMD:CP_Elec_10x10.5
- C3, C4: value 100n -> 100n,CX0805MRX7R7BB104
- D10: value D_Schottky -> 1N5824; footprint Diode_SMD:D_SOD-323_HandSoldering -> Diode_THT:D_5KPW_P12.70mm_Horizontal
- D11, D9: value D_Schottky -> D_Schottky,PMEG3030EP,115; footprint Diode_SMD:D_SOD-323_HandSoldering -> Diode_SMD:D_SOD-128
- D3: renamed from D5; value TVS -> TVS,VS15VUA1VWMTFTR; footprint Diode_SMD:D_SMA-SMB_Universal_Handsoldering -> Diode_SMD:D_TUMD2
- D4: renamed from D6; value Indicater -> LED,AP3216ID
- D6: renamed from D8; value D_Schottky -> D_Schottky,PMEG3030EP,115; footprint Diode_SMD:D_SOD-323_HandSoldering -> Diode_SMD:D_SOD-128
- F1: value Fuse(>15A) -> Fuse,CC12H15A-TR
- Q1, Q2: value IRLR7843 -> IRLML6344TRPBF; footprint Package_TO_SOT_SMD:TO-252-2 -> Package_TO_SOT_SMD:SOT-23
- R1, R4: value 100ohm -> 220 ohm,1/8W,RG2012P-221-B-T5
- R3, R5: value 1k -> 1k,SR0805FR-7W1KL
- R8: renamed from R10; value ~ -> 560ohm 1/2W,ERJ-UP6D5600V
- R9: renamed from R11; value ~ -> 180ohm 1/4W,CRCW0805180RFKEA
- renumbered 3s+1 to 3S, 2s+1 to 5V, GND1 to GND, H4 to H1, H3 to H2, H2 to H3, H1 to H4, J5 to J4, J4 to J5, J7 to J6, J6 to J7, R9 to R7
Connections:
- net 2sServo1: now also D7.1 (K); no longer D9.1 (K)
- net 3s+: now also D11.1 (K), C7.1, C9.1, D12.1 (K), Q3.1 (S), Q3.2 (S), Q3.3 (S), U1.1 (VIN); no longer C2.1
- net 3sMotor1: now also D9.1 (K); no longer D11.1 (K)
- net 3sMotor2: now also D8.1 (K); no longer D10.1 (K)
- net Backup_AV_FIRE: now also D9.2 (A); no longer D11.2 (A)
- net Backup_AV_PWM_Servo: now also D7.2 (A); no longer D9.2 (A)
- net GND: now also D10.1 (K), C7.2, C8.2, C9.2, D5.1 (K), U1.3 (GND), U1.5 (ON_OFF_N)
- net Main_AV_FIRE: now also D8.2 (A); no longer D10.2 (A)
- net at C3.1, J1.2 (Pin_2), Q1.1 (D): now also D11.2 (A)
- net at R7.1: now also Q3.4 (G)
- net at D3.2 (A2), F1.2: now also Q3.5 (D)
- net at C4.1, J2.2 (Pin_2), Q2.1 (D): now also D12.2 (A)
- net at R9.1: now also D5.2 (A)
- net 2s+ renamed 5V+
- net 5V+: now also C2.1, C8.1, L1.2, U1.4 (FEEDBACK)
- new net: D10.2 (A), L1.1, U1.2 (OUTPUT)
Other:
- note added: "5VBuck"
- note added: "5VServoMotor"
- note added: "D2防馬達斷電突波 C4防雜訊 C5防馬達啟動瞬間掉電壓"
- note added: "Q2(NMOS)作為開關 R5下拉電阻"
- note removed: "2sBuck"
- note removed: "2sServoMotor"
- note removed: "D7防馬達斷電突波 C1防雜訊 C2防馬達啟動瞬間掉電壓"
- note removed: "Q4(NMOS)作為開關 R3下拉電阻"

Commit message: Deployment Board
Parts:
- renumbered 3S to 3S1, 5V to 5V1, C5 to C2, C9 to C5, C2 to C6, D11 to D1, D12 to D2, GND to GND1, R3 to R2, R4 to R3, R5 to R4, R7 to R5, R8 to R6, R9 to R7
