File: Deployment board/Deployment board.kicad_pcb (KiCad board)
At the start: 4 copper layers, 57.1 x 54 mm, 52 parts, among them J1 Conn_01x02, J2 Conn_01x02, J3 Conn_01x02, J4 Conn_01x04, J5 Conn_01x04, J6 Conn_01x02, J7 Conn_01x02, M1 Motor_Servo, M2 Motor_Servo, Q1 IRLR7843, Q2 IRLR7843, Q3 FDD4141, U1 TPSM84824MOLR

Commit message: deployment board
Parts:
- removed C6: 1000u, Capacitor_SMD:CP_Elec_10x14.3
- removed D2: D_Schottky, Diode_SMD:D_SMA-SMB_Universal_Handsoldering
- removed the D4 at (55.6, 127.2)
- removed R12: 10k, Resistor_SMD:R_0805_2012Metric_Pad1.20x1.40mm_HandSolder
- removed R13: 866k, Resistor_SMD:R_0805_2012Metric_Pad1.20x1.40mm_HandSolder
- removed R14: 6.81k, Resistor_SMD:R_0805_2012Metric_Pad1.20x1.40mm_HandSolder
- removed R15: 34.8k, Resistor_SMD:R_0805_2012Metric_Pad1.20x1.40mm_HandSolder
- removed R2: 1k, Resistor_SMD:R_0805_2012Metric_Pad1.20x1.40mm_HandSolder
- removed the R7 at (50.7, 107.8)
- added D12: D_Schottky,PMEG3030EP,115, Diode_SMD:D_SOD-128, F.Cu at (222.2, 42.8)
- added D5: LED,AP3216ID, LED_SMD:LED_1206_3216Metric_Pad1.42x1.75mm_HandSolder, F.Cu at (222.2, 73.3)
- added D8: D_Schottky,PMEG3030EP,115, Diode_SMD:D_SOD-128, F.Cu at (223.2, 68.0)
- added L1: 33uH,SRN3010BTA-330M, Inductor_SMD_Wurth:L_Wurth_WE-LQSH-3012, F.Cu at (255.2, 31.2)
- C1, C2, C5: value 1000u -> 220uF,865060657012; footprint Capacitor_SMD:CP_Elec_10x14.3 -> Capacitor_SMD:CP_Elec_10x10.5
- C3, C4: value 100n -> 100n,CX0805MRX7R7BB104
- C7, C8: value 10uF 3.979mOhm -> 220uF,865060657012; footprint Capacitor_SMD:C_0805_2012Metric_Pad1.18x1.45mm_HandSolder -> Capacitor_SMD:CP_Elec_10x10.5
- C9: value 47uF 2.674mOhm Qty=3 -> 220uF,865060657012; footprint Capacitor_SMD:C_0805_2012Metric_Pad1.18x1.45mm_HandSolder -> Capacitor_SMD:CP_Elec_10x10.5
- D10: value D_Schottky -> 1N5824; footprint Diode_SMD:D_SOD-323_HandSoldering -> Diode_THT:D_5KPW_P12.70mm_Horizontal
- D11, D9: value D_Schottky -> D_Schottky,PMEG3030EP,115; footprint Diode_SMD:D_SOD-323_HandSoldering -> Diode_SMD:D_SOD-128
- D3: renamed from D5; value TVS -> TVS,VS15VUA1VWMTFTR; footprint Diode_SMD:D_SMA-SMB_Universal_Handsoldering -> Diode_SMD:D_TUMD2
- D4: renamed from D6; value Indicater -> LED,AP3216ID
- D6: renamed from D8; value D_Schottky -> D_Schottky,PMEG3030EP,115; footprint Diode_SMD:D_SOD-323_HandSoldering -> Diode_SMD:D_SOD-128
- D7: value Indicater -> D_Schottky,PMEG3030EP,115; footprint LED_SMD:LED_1206_3216Metric_Pad1.42x1.75mm_HandSolder -> Diode_SMD:D_SOD-128
- F1: value Fuse(>15A) -> Fuse,CC12H15A-TR
- Q1, Q2: value IRLR7843 -> IRLML6344TRPBF; footprint Package_TO_SOT_SMD:TO-252-2 -> Package_TO_SOT_SMD:SOT-23
- Q3: value FDD4141 -> SI7613DN-T1-GE3; footprint Package_TO_SOT_SMD:SOT-23 -> Package_SO:Vishay_PowerPAK_1212-8_Single
- R1, R4: value 100ohm -> 220 ohm,1/8W,RG2012P-221-B-T5
- R3, R5: value 1k -> 1k,SR0805FR-7W1KL
- R8: renamed from R10; value 3.3k -> 560ohm 1/2W,ERJ-UP6D5600V
- R9: renamed from R11; value 3.3k -> 180ohm 1/4W,CRCW0805180RFKEA
- U1: value TPSM84824MOLR -> LM2596S-5.0/NOPB; footprint TPSM84824:MOL0024A -> Package_TO_SOT_SMD:TO-263-5_TabPin3
- moved H3 242.7 mm to (261.2, 30.9)
- moved M1 216.9 mm to (258.6, 73.3), turned to -90 degrees
- moved M2 206.2 mm to (249.5, 73.3), turned to -90 degrees
- moved J6 197.1 mm to (248.7, 65.8), turned to 180 degrees
- moved C1 196.3 mm to (259.6, 63.5), turned to 180 degrees
- moved R5 193.0 mm to (222.6, 50.4)
- moved J7 192.2 mm to (238.9, 67.8), turned to 180 degrees
- moved C2 191.8 mm to (259.4, 51.8), turned to 180 degrees
- moved R4 191.3 mm to (230.7, 67.3), turned to -90 degrees
- moved C8 190.5 mm to (259.4, 40.2), turned to 180 degrees
- moved U1 190.3 mm to (246.7, 33.9), turned to 90 degrees
- moved J1 189.8 mm to (214.7, 47.1), turned to 90 degrees
- moved J2 189.5 mm to (214.7, 38.2), turned to 90 degrees
- moved C3 187.1 mm to (226.8, 47.1), turned to -90 degrees
- moved C5 184.9 mm to (234.9, 47.0), turned to 0 degrees
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- renumbered 3s+1 to 3S, 2s+1 to 5V, GND1 to GND, H4 to H1, H3 to H2, H2 to H3, H1 to H4, J5 to J4, J4 to J5, J7 to J6, J6 to J7, R9 to R7
Connections:
- 5V pad 1: 2s+ -> 5V+
- C1 pad 1: 2s+ -> 5V+
- C2 pad 1: 3s+ -> 5V+
- C3 pad 1: Net-(D2-A) -> Net-(D11-A)
- C8 pad 1: 3s+ -> 5V+
- C9 pad 1: 2s+ -> GND
- C9 pad 2: GND -> 3s+
- D10 pad 1: 3sMotor2 -> GND
- D10 pad 2: Main_AV_FIRE -> Net-(D10-A)
- D11 pad 1: 3sMotor1 -> 3s+
- D11 pad 2: Backup_AV_FIRE -> Net-(D11-A)
- D3 pad 2: Net-(D5-A2) -> Net-(D3-A2)
- D7 pad 1: GND -> 2sServo1
- D7 pad 2: Net-(D7-A) -> Backup_AV_PWM_Servo
- D9 pad 1: 2sServo1 -> 3sMotor1
- D9 pad 2: Backup_AV_PWM_Servo -> Backup_AV_FIRE
- F1 pad 2: Net-(D5-A2) -> Net-(D3-A2)
- J1 pad 2: Net-(D2-A) -> Net-(D11-A)
- M1 pad 2: 2s+ -> 5V+
- M2 pad 2: 2s+ -> 5V+
- Q1 pad 1: Net-(D2-A) -> Net-(D11-A)
- Q3 pad 1: Net-(Q3-G) -> 3s+
- Q3 pad 3: Net-(D5-A2) -> 3s+
- R9 pad 1: Net-(D7-A) -> Net-(D5-A)
- R9 pad 2: 2s+ -> 5V+
- U1 pad 1: 2s+ -> 3s+
- U1 pad 2: Net-(U1-FB) -> Net-(D10-A)
- U1 pad 4: unconnected-(U1-DNC-Pad4) -> 5V+
- U1 pad 5: Net-(U1-TT) -> GND
Routing:
- net 2s+: track 109.0 -> 0.00 mm, vias 2 -> 0
- net 5V+: track 0.00 -> 90.6 mm, vias 0 -> 5
- net 3sMotor1: track 70.0 -> 19.5 mm
- net 3s+: track 140.7 -> 108.2 mm, vias 0 -> 1
- net Net-(D11-A): track 0.00 -> 31.2 mm, vias 0 -> 1
- net Net-(D2-A): track 25.4 -> 0.00 mm
- net Net-(D10-A): track 0.00 -> 25.0 mm, vias 0 -> 1
- net 3sMotor2: track 43.9 -> 21.6 mm, vias 2 -> 3
- net Net-(D12-A): track 24.0 -> 41.4 mm, vias 0 -> 1
- net GND: track 89.7 -> 106.4 mm, vias 14 -> 11
- net 2sServo1: track 59.8 -> 44.7 mm
- net 2sServo2: track 55.8 -> 41.2 mm
- net Net-(U1-FB): track 9.45 -> 0.00 mm
- net Net-(D5-A2): track 8.87 -> 0.00 mm
- net Net-(Q1-G): track 14.2 -> 21.4 mm, vias 0 -> 2
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- added copper zone on In1.Cu, net 5V+
- removed copper zone on In1.Cu, net 2s+
Other:
- board size 57.1 x 54 mm -> 54.5 x 49 mm

Commit message: deployment board
Parts:
- moved J6 3.17 mm to (246.3, 68.0)
- moved D10 0.86 mm to (247.1, 60.6)
- moved C5 0.60 mm to (234.9, 46.4)
Routing:
- net 2sServo2: track 41.2 -> 36.2 mm
- net Net-(D10-A): track 25.0 -> 26.7 mm
- net 2sServo1: track 44.7 -> 45.3 mm
