File: SmallAvionic/Joyce2/SmallAvionic.kicad_pcb (KiCad board)
At the start: 4 copper layers, 74.9 x 94.8 mm, 103 parts, among them J1 Conn_01x02, J2 Boot_mode_pin, J3 Conn_01x04, J4 USB_C_Receptacle_USB2.0_16P, J5 Conn_01x03, J6 Conn_01x04, J7 Screw_Terminal_01x01, J8 Conn_01x03, Q1 TSM3481CX6 RFG, Q2 TSM3481CX6 RFG, Q3 NMOS, SW1 SW_Push, SW2 USER_Buttom, U1 LD1117S33TR_SOT223, U2 STM32F103C8Tx, U3 LTC4412xS6, U4 TPS54538RQFR, U5 MMC5983MA, U6 BMP390, U7 W25Q128JVS, U8 BMI088, Y1 8Mhz

Commit message: jpush
Parts:
- removed the R16 at (234.7, 103.0)
- added R16(PG_pull_up)1: 100k, Resistor_SMD:R_0805_2012Metric_Pad1.20x1.40mm_HandSolder, F.Cu at (225.2, 110.2)
- FB1: footprint LED_SMD:LED_0805_2012Metric_Pad1.15x1.40mm_HandSolder -> Inductor_SMD:L_0805_2012Metric_Pad1.05x1.20mm_HandSolder
- R9: footprint Inductor_SMD:L_0805_2012Metric_Pad1.05x1.20mm_HandSolder -> Resistor_SMD:R_0805_2012Metric_Pad1.20x1.40mm_HandSolder
- SW1, SW2: footprint Button_Switch_SMD:SW_Push_1P1T_NO_CK_PTS125Sx43PSMTR -> Button_Switch_SMD:SW_Push_1P1T_NO_E-Switch_TL3301NxxxxxG
- moved J7 50.7 mm to (202.6, 65.5), turned to -90 degrees
- moved C4 43.9 mm to (207.8, 91.1)
- moved C30 42.9 mm to (207.8, 93.6)
- moved C25 34.2 mm to (207.8, 88.9)
- moved R26 22.5 mm to (211.3, 74.2), turned to 180 degrees
- moved D5 20.2 mm to (208.4, 97.2), turned to 90 degrees
- moved Q3 20.1 mm to (202.0, 104.8)
- moved SW2 19.8 mm to (201.9, 93.2), turned to 90 degrees
- moved R21 19.1 mm to (207.3, 74.3)
- moved R25 19.0 mm to (208.1, 100.8)
- moved D4 18.7 mm to (211.3, 97.2), turned to 90 degrees
- moved SW1 17.6 mm to (201.8, 81.2), turned to 90 degrees
- moved D6 13.8 mm to (207.9, 109.6)
- moved R24 13.8 mm to (214.7, 102.2)
- moved R28 13.8 mm to (214.8, 104.5)
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Routing:
- net GND: track 150.7 -> 319.4 mm, vias 7 -> 12
- net +3.3V: track 107.6 -> 265.5 mm, vias 6 -> 11
- net V_BAT+: track 42.4 -> 142.4 mm, vias 1 -> 2
- net USART1_RX: track 4.90 -> 54.6 mm
- net USART1_TX: track 4.43 -> 53.4 mm
- net Buzzer: track 2.98 -> 48.9 mm, vias 1 -> 2
- net I2C1_SDA: track 11.3 -> 54.6 mm
- net NRST: track 2.11 -> 41.5 mm, vias 1 -> 2
- net USER_BT: track 0.00 -> 37.9 mm, vias 0 -> 2
- net I2C1_SCL: track 10.2 -> 44.5 mm, vias 2 -> 3
- net LED_State: track 1.52 -> 26.8 mm, vias 1 -> 2
- net Net-(D3-A): track 26.8 -> 2.35 mm, vias 2 -> 0
- net LED_SYS: track 1.69 -> 24.9 mm, vias 1 -> 2
- net +USB_5V: track 13.1 -> 35.7 mm
- net Net-(BZ1--): track 14.4 -> 28.6 mm
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Other:
- board size 74.9 x 94.8 mm -> 58.2 x 76.6 mm
