File: SmallAvionic/Joyce2/SmallAvionic.kicad_sch (KiCad schematic)
At the start: 103 parts, among them J1 Conn_01x02, J2 Boot_mode_pin, J3 Conn_01x04, J4 USB_C_Receptacle_USB2.0_16P, J5 Conn_01x03, J6 Conn_01x04, J7 Screw_Terminal_01x01, J8 Conn_01x03, Q1 TSM3481CX6 RFG, Q2 TSM3481CX6 RFG, Q3 NMOS, SW1 SW_Push, SW2 USER_Buttom, U1 LD1117S33TR_SOT223, U2 STM32F103C8Tx, U3 LTC4412xS6, U4 TPS54538RQFR, U5 MMC5983MA, U6 BMP390, U7 W25Q128JVS, U8 BMI088, Y1 8Mhz

Commit message: jpush
Parts:
- BZ1: footprint (none) -> Buzzer_Beeper:Buzzer_15x7.5RM7.6
- D1: footprint (none) -> Diode_SMD:D_SMA-SMB_Universal_Handsoldering
- D2, D3, D4, D5, FB1: footprint (none) -> LED_SMD:LED_0805_2012Metric_Pad1.15x1.40mm_HandSolder
- F1: footprint (none) -> Fuse:Fuse_1206_3216Metric_Pad1.42x1.75mm_HandSolder
- J1: footprint (none) -> Connector_Molex:Molex_Micro-Fit_3.0_43650-0221_1x02_P3.00mm_Vertical
- J2: footprint (none) -> Connector_PinSocket_2.00mm:PinSocket_1x02_P2.00mm_Vertical
- J3: footprint (none) -> Connector_PinSocket_2.00mm:PinSocket_1x04_P2.00mm_Vertical
- J4: footprint (none) -> Connector_USB:USB_C_Receptacle_HCTL_HC-TYPE-C-16P-01A
- J6: footprint (none) -> Connector_JST:JST_EH_B4B-EH-A_1x04_P2.50mm_Vertical
- J7: footprint (none) -> TerminalBlock_MetzConnect:TerminalBlock_MetzConnect_360271_1x01_Horizontal_ScrewM3.0_Boxed
- J8: footprint (none) -> Connector_JST:JST_GH_BM03B-GHS-TBT_1x03-1MP_P1.25mm_Vertical
- L1, R16(PG_pull_up)1, R9: footprint (none) -> Inductor_SMD:L_0805_2012Metric_Pad1.05x1.20mm_HandSolder
- Q3: footprint (none) -> Package_TO_SOT_SMD:TO-252-2
- R1, R10, R11, R12, R13, R14, R15, R16, R17, R18, R19, R2, R20, R21, R22, R23, R24, R25, R26, R27, R28, R29, R3, R30, R31, R32, R4, R40, R5, R6, R7, R8: footprint (none) -> Resistor_SMD:R_0805_2012Metric_Pad1.20x1.40mm_HandSolder
- SW1, SW2: footprint (none) -> Button_Switch_SMD:SW_Push_1P1T_NO_CK_PTS125Sx43PSMTR
- U4: footprint VQFN-HR9_RQF_TEX -> Small_av_joyce_lib:VQFN-HR9_RQF_TEX
- U5: footprint MMC5983MA_MEM -> Small_av_joyce_lib:MMC5983MA_MEM
- U6: footprint 10LGA_2X2X0p75_BOS -> Small_av_joyce_lib:10LGA_2X2X0p75_BOS
- Y1: footprint (none) -> Crystal:Crystal_SMD_0603-4Pin_6.0x3.5mm_HandSoldering; private KLC_S4.1 -> (none)
Connections:
- no-connect marks 4 -> 6
Other:
- removed sheet Deployment Board

Commit message: jpush
Parts:
- FB1: footprint LED_SMD:LED_0805_2012Metric_Pad1.15x1.40mm_HandSolder -> Inductor_SMD:L_0805_2012Metric_Pad1.05x1.20mm_HandSolder
- R16(PG_pull_up)1, R9: footprint Inductor_SMD:L_0805_2012Metric_Pad1.05x1.20mm_HandSolder -> Resistor_SMD:R_0805_2012Metric_Pad1.20x1.40mm_HandSolder
- SW1, SW2: footprint Button_Switch_SMD:SW_Push_1P1T_NO_CK_PTS125Sx43PSMTR -> Button_Switch_SMD:SW_Push_1P1T_NO_E-Switch_TL3301NxxxxxG
Changed lines of the file:
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@@
 			)
 		)
-		(property "Footprint" "Inductor_SMD:L_0805_2012Metric_Pad1.05x1.20mm_HandSolder"
+		(property "Footprint" "Resistor_SMD:R_0805_2012Metric_Pad1.20x1.40mm_HandSolder"
 			(at 144.78 347.218 90)
 			(effects
@@
 			)
 		)
-		(property "Footprint" "Button_Switch_SMD:SW_Push_1P1T_NO_CK_PTS125Sx43PSMTR"
+		(property "Footprint" "Button_Switch_SMD:SW_Push_1P1T_NO_E-Switch_TL3301NxxxxxG"
 			(at 312.42 337.82 0)
 			(effects
@@
 			)
 		)
-		(property "Footprint" "Inductor_SMD:L_0805_2012Metric_Pad1.05x1.20mm_HandSolder"
+		(property "Footprint" "Resistor_SMD:R_0805_2012Metric_Pad1.20x1.40mm_HandSolder"
 			(at 109.22 231.902 90)
 			(effects
@@
 		(exclude_from_sim no)
 		(in_bom yes)
-		(on_board no)
+		(on_board yes)
 		(dnp no)
 		(fields_autoplaced yes)
@@
 			)
 		)
-		(property "Footprint" "LED_SMD:LED_0805_2012Metric_Pad1.15x1.40mm_HandSolder"
+		(property "Footprint" "Inductor_SMD:L_0805_2012Metric_Pad1.05x1.20mm_HandSolder"
 			(at 123.19 48.768 90)
 			(effects
@@
 			)
 		)
-		(property "Footprint" "Button_Switch_SMD:SW_Push_1P1T_NO_CK_PTS125Sx43PSMTR"
+		(property "Footprint" "Button_Switch_SMD:SW_Push_1P1T_NO_E-Switch_TL3301NxxxxxG"
 			(at 33.02 92.71 0)
 			(effects
