File: BigAvionic/Second_layer_MCU/Second_layer_MCU.kicad_pcb (KiCad board)
At the start: 4 copper layers, 68 x 68 mm, 98 parts, among them J1 Conn_01x04, J10 Conn_01x04, J11 Conn_01x04, J13 Conn_01x08, J14 Conn_01x08, J2 USB_C_Receptacle_USB2.0_16P, J3 Conn_01x02, J4 Micro_SD_Card_Det1, J5 Conn_01x04, J6 Conn_01x04, J7 Screw_Terminal_01x02, J8 Conn_01x04, J9 Conn_01x08, Q2 BSS138, SW1 SW_Push, SW2 USER_Buttom, SW3 USER_Buttom, U1 STM32F405VGTx, U2 W25Q128JVS, U3 ADXL375BCCZ, U4 BMP390, U5 BMI088, Y1 8Mhz

Commit message: Big av slight modification+add libraries folder
Parts:
- C17, C18: value 22pF -> 15pF
- SW2, SW3: value USER_Buttom -> SW_Push_Shielded
- Y1: value 8Mhz -> FA-238 16Mhz; footprint Crystal:Crystal_SMD_3225-4Pin_3.2x2.5mm_HandSoldering -> Crystal:Crystal_SMD_SeikoEpson_FA238-4Pin_3.2x2.5mm
- moved R5 1.33 mm to (107.1, 115.4)
- moved SW2 0.21 mm to (107.0, 125.5)
Routing:
- net GND: track 93.9 -> 92.6 mm, vias 120 -> 217
- net UART6_RX: track 35.2 -> 34.2 mm
Other:
- board text added: "3V3"
- board text added: "GND"
- board text added: "I2C1_SCL"
- board text added: "I2C1_SDA"
